Commit message: まずURDFが正常なとき

File: leg_l/leg_l.urdf.xacro (robot description, xacro)
@@ -193,5 +193,5 @@
 	    	<axis xyz="0 -1 0"/>
 	    	<limit effort="1000.0" lower="-3.141593" upper="3.141593" velocity="0.5"/>
-	    	<mimic joint="${name}_joint4" multiplier="1" offset="0"/>
+	    	<!-- <mimic joint="${name}_joint4" multiplier="1" offset="0"/>  -->
 	  	</joint>
 		<!-- toe -->
