Commit message: 開いたSDFをサーボで動かせた

File: urdf/simple_open_chain.urdf (robot description, URDF)
Before this commit: robot closed_chain, 4 links, 3 joints
Links:
- removed link closed_chain_right_pad1
- removed link closed_chain_right_pad2
- removed link closed_chain_right_pad3
- removed link closed_chain_right_pad4
- added link right_pad1, mass 1.41502697; collision box size=1.0 1.0 0.1; visual box size=1.0 1.0 0.1
- added link right_pad2, mass 1.41502697; collision box size=1.0 1.0 0.1; visual box size=1.0 1.0 0.1
- added link right_pad3, mass 1.41502697; collision box size=1.0 1.0 0.1; visual box size=1.0 1.0 0.1
- added link right_pad4, mass 1.41502697; collision box size=1.0 1.0 0.1; visual box size=1.0 1.0 0.1
Joints:
- removed joint closed_chain_right_pad_joint1
- removed joint closed_chain_right_pad_joint2
- removed joint closed_chain_right_pad_joint3
- added joint right_pad_joint1: type revolute, parent right_pad1, child right_pad2, origin xyz=1  0  0 rpy=0  0  0, axis 0  1  0, limit lower=-3.14 upper=3.14 effort=100 velocity=10.
- added joint right_pad_joint2: type revolute, parent right_pad2, child right_pad3, origin xyz=1  0  0 rpy=0  0  0, axis 0  1  0, limit lower=-3.14 upper=3.14 effort=100 velocity=10.
- added joint right_pad_joint3: type revolute, parent right_pad3, child right_pad4, origin xyz=1  0  0 rpy=0  0  0, axis 0  1  0, limit lower=-3.14 upper=3.14 effort=100 velocity=10.
