Commit message: 見やすくするため、ひとつ目のリンクを太くした

File: xacro/01_open_chain.xacro (robot description, xacro)
@@ -15,13 +15,13 @@
   <link name="right_pad1">
     <collision name="right_pad1_collision">
-      <origin xyz="0.5 0 0" rpy="0 0 0"/>
+      <origin xyz="0.5 0 0.25" rpy="0 0 0"/>
       <geometry>
-        <box size="1.0 1.0 0.1" />
+        <box size="1.0 1.0 0.5" />
       </geometry>
     </collision>
     <visual name="right_pad1_visual">
-      <origin xyz="0.5 0 0" rpy="0 0 0"/>
+      <origin xyz="0.5 0 0.25" rpy="0 0 0"/>
       <geometry>
-        <box size="1.0 1.0 0.1" />
+        <box size="1.0 1.0 0.5" />
       </geometry>
       <material name="red"/>
@@ -41,5 +41,5 @@
     <parent link="right_pad1"/>
     <child  link="right_pad2"/>
-    <origin xyz="1.0 0 0" rpy="0 -1.57 0"/>
+    <origin xyz="1.0 0 0.5" rpy="0 -1.57 0"/>
     <axis xyz="0 1 0"/>
     <limit effort="1000.0" lower="-3.14" upper="3.14" velocity="1000.0"/>
@@ -48,5 +48,5 @@
   <link name="right_pad2">
     <collision name="right_pad2_collision">
-      <origin xyz="0.5 0 0" rpy="0 0 0"/>
+      <origin xyz="0.5 0 -0.05" rpy="0 0 0"/>
       <geometry>
         <box size="1.0 1.0 0.1" />
@@ -54,5 +54,5 @@
     </collision>
     <visual name="right_pad2_visual">
-      <origin xyz="0.5 0 0" rpy="0 0 0"/>
+      <origin xyz="0.5 0 -0.05" rpy="0 0 0"/>
       <geometry>
         <box size="1.0 1.0 0.1" />
@@ -79,5 +79,5 @@
   <link name="right_pad3">
     <collision name="right_pad3_collision">
-      <origin xyz="0.5 0 0" rpy="0 0 0"/>
+      <origin xyz="0.5 0 -0.05" rpy="0 0 0"/>
       <geometry>
         <box size="1.0 1.0 0.1" />
@@ -85,5 +85,5 @@
     </collision>
     <visual name="right_pad3_visual">
-      <origin xyz="0.5 0 0" rpy="0 0 0"/>
+      <origin xyz="0.5 0 -0.05" rpy="0 0 0"/>
       <geometry>
         <box size="1.0 1.0 0.1" />
@@ -110,5 +110,5 @@
   <link name="right_pad4">
     <collision name="right_pad4_collision">
-      <origin xyz="0.5 0 0" rpy="0 0 0"/>
+      <origin xyz="0.5 0 -0.05" rpy="0 0 0"/>
       <geometry>
         <box size="1.0 1.0 0.1" />
@@ -116,5 +116,5 @@
     </collision>
     <visual name="right_pad4_visual">
-      <origin xyz="0.5 0 0" rpy="0 0 0"/>
+      <origin xyz="0.5 0 -0.05" rpy="0 0 0"/>
       <geometry>
         <box size="1.0 1.0 0.1" />
