Commit message: Add xacro for pegasus gazebo plugin

File: xacro/02_open_chain_and_dummy_link.xacro (robot description, xacro)
@@ -13,12 +13,15 @@
     <color rgba="1.0 1.0 0.0 1.0"/>
   </material>
+  <xacro:macro name="box_inertial" params="mass origin d w h">
+    <inertial>
+      <origin xyz="${origin}" rpy="0 0 0"/>
+      <mass value="${mass}"/>
+      <inertia ixx="${mass * (w ** 2 + h ** 2) / 12}"
+               ixy="0.0" iyy="${mass * (d ** 2 + h ** 2) / 12}"
+               ixz="0.0" iyz="0.0" izz="${mass * (w ** 2 + d ** 2) / 12}"/>
+    </inertial>
+  </xacro:macro>
   <link name="right_pad1">
-    <collision name="right_pad1_collision">
-      <origin xyz="0.5 0 0.25" rpy="0 0 0"/>
-      <geometry>
-        <box size="1.0 1.0 0.5" />
-      </geometry>
-    </collision>
-    <visual name="right_pad1_visual">
+    <visual>
       <origin xyz="0.5 0 0.25" rpy="0 0 0"/>
       <geometry>
@@ -27,13 +30,23 @@
       <material name="red"/>
     </visual>
-    <inertial>
-      <mass value="0.5"/>
+    <collision>
       <origin xyz="0.5 0 0.25" rpy="0 0 0"/>
-      <inertia
-        ixx="0.0001"
-        ixy="0.0000" iyy="0.0001"
-        ixz="0.0000" iyz="0.0000" izz="0.0001"/>
-    </inertial>
+      <geometry>
+        <box size="1.0 1.0 0.5" />
+      </geometry>
+    </collision>
+    <xacro:box_inertial mass="0.5" origin="0.5 0 0.25" d="1.0" w="1.0" h="0.5"/>
   </link>
+  <gazebo reference="right_pad1">
+    <material>Gazebo/Red</material>
+    <mu1>100000</mu1>
+    <mu2>100000</mu2>
+    <kp>40000.0</kp>
+    <kd>0.0</kd>
+    <minDepth>0.0</minDepth>
+    <maxContacts>5</maxContacts>
+    <selfCollide>false</selfCollide>
+    <dampingFactor>0.0</dampingFactor>
+  </gazebo>
   <!-- Joints are respect the PARENT in XACRO/URDF -->
   <!-- Joints are respect the CHILD in SDF -->
@@ -60,13 +73,17 @@
       <material name="green"/>
     </visual>
-    <inertial>
-      <mass value="0.5"/>
-      <origin xyz="0.5 0 -0.05" rpy="0 0 0"/>
-      <inertia
-        ixx="0.0001"
-        ixy="0.0000" iyy="0.0001"
-        ixz="0.0000" iyz="0.0000" izz="0.0001"/>
-    </inertial>
+    <xacro:box_inertial mass="0.5" origin="0.5 0 -0.05" d="1.0" w="1.0" h="0.1"/>
   </link>
+  <gazebo reference="right_pad2">
+    <material>Gazebo/Green</material>
+    <mu1>100000</mu1>
+    <mu2>100000</mu2>
+    <kp>40000.0</kp>
+    <kd>0.0</kd>
+    <minDepth>0.0</minDepth>
+    <maxContacts>5</maxContacts>
+    <selfCollide>false</selfCollide>
+    <dampingFactor>0.0</dampingFactor>
+  </gazebo>
   <joint name="right_pad2_joint" type="revolute">
     <parent link="right_pad2"/>
@@ -91,13 +108,17 @@
       <material name="blue"/>
     </visual>
-    <inertial>
-      <mass value="0.5"/>
-      <origin xyz="0.5 0 -0.05" rpy="0 0 0"/>
-      <inertia
-        ixx="0.0001"
-        ixy="0.0000" iyy="0.0001"
-        ixz="0.0000" iyz="0.0000" izz="0.0001"/>
-    </inertial>
+    <xacro:box_inertial mass="0.5" origin="0.5 0 -0.05" d="1.0" w="1.0" h="0.1"/>
   </link>
+  <gazebo reference="right_pad3">
+    <material>Gazebo/Blue</material>
+    <mu1>100000</mu1>
+    <mu2>100000</mu2>
+    <kp>40000.0</kp>
+    <kd>0.0</kd>
+    <minDepth>0.0</minDepth>
+    <maxContacts>5</maxContacts>
+    <selfCollide>false</selfCollide>
+    <dampingFactor>0.0</dampingFactor>
+  </gazebo>
   <joint name="right_pad3_joint" type="revolute">
     <parent link="right_pad3"/>
@@ -122,13 +143,17 @@
       <material name="yellow"/>
     </visual>
-    <inertial>
-      <mass value="0.5"/>
-      <origin xyz="0.5 0 -0.05" rpy="0 0 0"/>
-      <inertia
-        ixx="0.0001"
-        ixy="0.0000" iyy="0.0001"
-        ixz="0.0000" iyz="0.0000" izz="0.0001"/>
-    </inertial>
+    <xacro:box_inertial mass="0.5" origin="0.5 0 -0.05" d="1.0" w="1.0" h="0.1"/>
   </link>
+  <gazebo reference="right_pad4">
+    <material>Gazebo/Yellow</material>
+    <mu1>100000</mu1>
+    <mu2>100000</mu2>
+    <kp>40000.0</kp>
+    <kd>0.0</kd>
+    <minDepth>0.0</minDepth>
+    <maxContacts>5</maxContacts>
+    <selfCollide>false</selfCollide>
+    <dampingFactor>0.0</dampingFactor>
+  </gazebo>
   <!-- This joint closes the loop. -->
   <joint name="connection_joint" type="continuous">

File: xacro/04_pegasus.xacro (robot description, xacro)
@@ -1,4 +1,4 @@
-<?xml version="1.0"?>
-<robot name="incorrect_xacro" xmlns:xacro="http://www.ros.org/wiki/xacro">
+<?xml version="1.0" encoding="UTF-8"?>
+<robot name="test_robot_01" xmlns:xacro="http://www.ros.org/wiki/xacro">
   <material name="red">
     <color rgba="1.0 0.0 0.0 1.0"/>
@@ -156,3 +156,12 @@
     <dampingFactor>0.0</dampingFactor>
   </gazebo>
+<!--   <gazebo>
+    <plugin name="Myrobot_ClosedLoopPlugin" filename="libpegasus_gazebo_closed_loop_plugin.so">
+       <joint>add_joint</joint>
+       <child>right_pad1</child>
+       <parent>right_pad4</parent>
+       <position>1.0 0.0 0.0</position>
+       <rotation>0.0 0.0 0.0</rotation>
+    </plugin>
+  </gazebo> -->
 </robot>
